File: 20A Motor Controller.brd (EAGLE design)
At the start: 57.1 x 77.1 mm, 28 parts, among them IC1 BTN8962TA, IC2 BTN8962TA, Q1 FDD4141TO252

Commit message: Add files via upload
Parts:
- moved R3 3.40 mm to (58.0, 24.6)
Routing:
- net SR1: track 20.1 -> 15.6 mm
- net INH_PIN: track 7.85 -> 9.21 mm
- net INH: track 56.2 -> 55.0 mm
Changed lines of the file:
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@@
 <text x="58.039" y="51.181" size="0.8128" layer="22" font="vector" rot="MR0">H</text>
 <text x="60.579" y="51.181" size="0.8128" layer="22" font="vector" rot="MR0">H</text>
-<wire x1="61.595" y1="58.547" x2="55.626" y2="58.547" width="0.0762" layer="22"/>
+<wire x1="61.595" y1="58.547" x2="54.102" y2="58.547" width="0.0762" layer="22"/>
 <text x="55.372" y="55.372" size="0.8128" layer="22" font="vector" rot="MR0">L</text>
 <text x="58.039" y="53.975" size="0.8128" layer="22" font="vector" rot="MR0">L</text>
@@
 <attribute name="NAME" x="57.289" y="17.76" size="1.778" layer="25" font="vector" ratio="15" rot="R270"/>
 </element>
-<element name="R3" library="rcl" library_urn="urn:adsk.eagle:library:334" package="R0805" value="10K" x="58.039" y="21.209" smashed="yes" rot="R270">
-<attribute name="NAME" x="57.404" y="23.368" size="0.8128" layer="25" font="vector"/>
-<attribute name="VALUE" x="59.182" y="23.241" size="0.8128" layer="27" rot="R270"/>
+<element name="R3" library="rcl" library_urn="urn:adsk.eagle:library:334" package="R0805" value="10K" x="57.9882" y="24.6126" smashed="yes" rot="R270">
+<attribute name="NAME" x="57.3532" y="26.7716" size="0.8128" layer="25" font="vector"/>
+<attribute name="VALUE" x="59.1312" y="26.6446" size="0.8128" layer="27" rot="R270"/>
 </element>
 <element name="R4" library="rcl" library_urn="urn:adsk.eagle:library:334" package="R0805" value="10K" x="61.468" y="31.369" smashed="yes" rot="R180">
@@
 <via x="78.232" y="42.926" extent="1-16" drill="0.45"/>
 <via x="78.232" y="40.767" extent="1-16" drill="0.45"/>
+<via x="60.9854" y="67.4878" extent="1-16" drill="0.45"/>
+<via x="62.103" y="67.4878" extent="1-16" drill="0.45"/>
+<via x="63.246" y="67.4878" extent="1-16" drill="0.45"/>
+<via x="64.3636" y="67.4878" extent="1-16" drill="0.45"/>
+<via x="61.4934" y="66.5734" extent="1-16" drill="0.45"/>
+<via x="62.6364" y="66.548" extent="1-16" drill="0.45"/>
+<via x="63.8302" y="66.548" extent="1-16" drill="0.45"/>
+<via x="64.135" y="24.003" extent="1-16" drill="0.45"/>
+<via x="65.151" y="24.003" extent="1-16" drill="0.45"/>
+<via x="66.167" y="24.003" extent="1-16" drill="0.45"/>
+<via x="64.135" y="22.987" extent="1-16" drill="0.45"/>
+<via x="65.151" y="22.987" extent="1-16" drill="0.45"/>
+<via x="66.167" y="22.987" extent="1-16" drill="0.45"/>
 </signal>
 <signal name="OUT1" class="2">
@@
 <contactref element="INPUT" pad="2"/>
 <contactref element="R3" pad="2"/>
-<wire x1="51.054" y1="18.161" x2="55.941" y2="18.161" width="0.3048" layer="1"/>
-<wire x1="55.941" y1="18.161" x2="58.039" y2="20.259" width="0.3048" layer="1"/>
+<wire x1="51.054" y1="18.161" x2="52.4866" y2="18.161" width="0.3048" layer="1"/>
+<wire x1="52.4866" y1="18.161" x2="57.9882" y2="23.6626" width="0.3048" layer="1"/>
 </signal>
 <signal name="IN1_PIN">
@@
 <contactref element="INPUT" pad="3"/>
 <contactref element="R5" pad="2"/>
-<wire x1="51.054" y1="23.241" x2="54.549" y2="23.241" width="0.3048" layer="1"/>
-<wire x1="54.549" y1="23.241" x2="60.518" y2="29.21" width="0.3048" layer="1"/>
+<wire x1="56.642" y1="27.3812" x2="58.674" y2="27.3812" width="0.3048" layer="1"/>
+<wire x1="58.674" y1="27.3812" x2="59.436" y2="28.1432" width="0.3048" layer="1"/>
+<wire x1="59.436" y1="28.1432" x2="60.518" y2="29.21" width="0.3048" layer="1"/>
+<wire x1="51.054" y1="23.241" x2="52.5018" y2="23.241" width="0.3048" layer="1"/>
+<wire x1="52.5018" y1="23.241" x2="56.642" y2="27.3812" width="0.3048" layer="1"/>
 </signal>
 <signal name="IS">
@@
 <contactref element="R2" pad="1"/>
 <contactref element="C7" pad="1"/>
-<wire x1="68.6235" y1="61.336" x2="64.902" y2="61.336" width="0.3048" layer="1"/>
-<wire x1="64.902" y1="61.336" x2="64.643" y2="61.595" width="0.3048" layer="1"/>
-<wire x1="64.643" y1="61.595" x2="64.643" y2="63.5" width="0.3048" layer="1"/>
-<wire x1="64.643" y1="63.5" x2="64.135" y2="64.008" width="0.3048" layer="1"/>
-<wire x1="64.135" y1="64.008" x2="61.087" y2="64.008" width="0.3048" layer="1"/>
-<wire x1="61.087" y1="64.008" x2="60.5402" y2="64.5548" width="0.3048" layer="1"/>
-<wire x1="60.5402" y1="64.5548" x2="60.5402" y2="70.6122" width="0.3048" layer="1"/>
-<wire x1="60.5402" y1="70.6122" x2="61.468" y2="71.54" width="0.3048" layer="1"/>
 <wire x1="61.468" y1="71.54" x2="63.527" y2="71.54" width="0.3048" layer="1"/>
-<wire x1="63.527" y1="71.54" x2="63.627" y2="71.44" width="0.4064" layer="1"/>
+<wire x1="63.627" y1="71.44" x2="63.527" y2="71.54" width="0.4064" layer="1"/>
+<wire x1="68.6235" y1="61.336" x2="68.0583" y2="61.9012" width="0.3048" layer="1"/>
+<wire x1="68.0583" y1="61.9012" x2="65.9108875" y2="61.9012" width="0.3048" layer="1"/>
+<wire x1="65.9108875" y1="61.9012" x2="65.357" y2="62.4550875" width="0.3048" layer="1"/>
+<wire x1="65.357" y1="69.71" x2="63.627" y2="71.44" width="0.3048" layer="1"/>
+<wire x1="65.357" y1="62.4550875" x2="65.357" y2="69.71" width="0.3048" layer="1"/>
 </signal>
 <signal name="SR2">
@@
 <contactref element="IC2" pad="3"/>
 <contactref element="R3" pad="1"/>
-<wire x1="58.039" y1="22.159" x2="58.039" y2="22.479" width="0.3048" layer="1"/>
-<wire x1="58.039" y1="22.479" x2="60.833" y2="25.273" width="0.3048" layer="1"/>
-<wire x1="63.627" y1="25.273" x2="60.833" y2="25.273" width="0.3048" layer="1"/>
+<wire x1="60.833" y1="25.273" x2="63.627" y2="25.273" width="0.3048" layer="1"/>
 <wire x1="63.627" y1="25.273" x2="68.5325" y2="25.273" width="0.3048" layer="1"/>
 <wire x1="68.5325" y1="25.273" x2="68.5985" y2="25.207" width="0.3048" layer="1"/>
 <wire x1="68.6235" y1="63.876" x2="67.051" y2="63.876" width="0.3048" layer="1"/>
-<wire x1="67.051" y1="63.876" x2="66.04" y2="62.865" width="0.3048" layer="1"/>
-<wire x1="66.04" y1="62.865" x2="66.04" y2="62.738" width="0.3048" layer="1"/>
-<via x="66.04" y="62.738" extent="1-16" drill="0.35"/>
-<wire x1="66.04" y1="62.738" x2="65.786" y2="62.611" width="0.3048" layer="16"/>
-<wire x1="65.786" y1="62.611" x2="62.357" y2="59.182" width="0.3048" layer="16"/>
+<wire x1="67.051" y1="63.876" x2="66.2432" y2="63.0682" width="0.3048" layer="1"/>
+<wire x1="66.2432" y1="63.0682" x2="66.2432" y2="62.7888" width="0.3048" layer="1"/>
+<via x="66.2432" y="62.7888" extent="1-16" drill="0.35"/>
+<wire x1="66.2432" y1="62.7888" x2="65.9384" y2="62.7888" width="0.3048" layer="16"/>
+<wire x1="65.9384" y1="62.7888" x2="62.357" y2="59.182" width="0.3048" layer="16"/>
 <wire x1="62.357" y1="59.182" x2="62.357" y2="47.752" width="0.3048" layer="16"/>
 <wire x1="62.357" y1="47.752" x2="65.405" y2="44.704" width="0.3048" layer="16"/>
@@
 <via x="63.627" y="26.543" extent="1-16" drill="0.35"/>
 <wire x1="63.627" y1="26.543" x2="63.627" y2="25.273" width="0.3048" layer="1"/>
+<wire x1="57.9882" y1="25.5626" x2="60.5434" y2="25.5626" width="0.3048" layer="1"/>
+<wire x1="60.5434" y1="25.5626" x2="60.833" y2="25.273" width="0.3048" layer="1"/>
 </signal>
 <signal name="IN1">
 <contactref element="IC1" pad="2"/>
 <contactref element="R4" pad="1"/>
-<wire x1="68.6235" y1="65.146" x2="65.527" y2="65.146" width="0.3048" layer="1"/>
-<via x="65.278" y="64.897" extent="1-16" drill="0.35"/>
-<wire x1="65.278" y1="64.897" x2="65.278" y2="62.9419125" width="0.3048" layer="16"/>
+<wire x1="68.6235" y1="65.146" x2="66.797" y2="65.146" width="0.3048" layer="1"/>
+<via x="66.294" y="65.151" extent="1-16" drill="0.35"/>
+<wire x1="66.294" y1="65.151" x2="66.294" y2="63.9572" width="0.3048" layer="16"/>
+<wire x1="66.294" y1="63.9572" x2="65.2787125" y2="62.9419125" width="0.3048" layer="16"/>
+<wire x1="65.2787125" y1="62.9419125" x2="65.278" y2="62.9419125" width="0.3048" layer="16"/>
 <wire x1="65.278" y1="62.9419125" x2="61.8998" y2="59.5637125" width="0.3048" layer="16"/>
 <wire x1="61.8998" y1="47.56261875" x2="64.9478" y2="44.51461875" width="0.3048" layer="16"/>
@@
 <wire x1="64.135" y1="33.528" x2="64.135" y2="33.086" width="0.3048" layer="1"/>
 <wire x1="64.135" y1="33.086" x2="62.418" y2="31.369" width="0.3048" layer="1"/>
-<wire x1="65.527" y1="65.146" x2="65.278" y2="64.897" width="0.3048" layer="1"/>
+<wire x1="66.797" y1="65.146" x2="66.294" y2="65.151" width="0.3048" layer="1"/>
 <wire x1="61.8998" y1="59.5637125" x2="61.8998" y2="47.56261875" width="0.3048" layer="16"/>
 <wire x1="64.9478" y1="44.51461875" x2="64.9478" y2="34.2138" width="0.3048" layer="16"/>

Commit message: Add files via upload
Parts:
- removed C14, C2: 470uf, rcl:E2,5-6
- removed D1: 10V, diode:SOT23
- added C11: 470uf, adafruit:TT5D10
- added D2: 39v, diode:SMB
Connections:
- net GND: now also C11.-; no longer C13.2, C14.-, C2.-
- net Q1_GATE: now also D2.A; no longer D1.1
- net V+: now also C11.+, D2.C; no longer C14.+, C2.+, D1.3
Changed lines of the file:
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@@
 </class>
 </classes>
-<designrules name="default">
+<designrules name="default *">
 <description language="de">&lt;b&gt;EAGLE Design Rules&lt;/b&gt;
 &lt;p&gt;
@@
 design rules under a new name.</description>
 <param name="layerSetup" value="(1*16)"/>
-<param name="mtCopper" value="0.035mm 0.035mm 0.035mm 0.035mm 0.035mm 0.035mm 0.035mm 0.035mm 0.035mm 0.035mm 0.035mm 0.035mm 0.035mm 0.035mm 0.035mm 0.035mm"/>
+<param name="mtCopper" value="0.07mm 0.035mm 0.035mm 0.035mm 0.035mm 0.035mm 0.035mm 0.035mm 0.035mm 0.035mm 0.035mm 0.035mm 0.035mm 0.035mm 0.035mm 0.07mm"/>
 <param name="mtIsolate" value="1.5mm 0.15mm 0.2mm 0.15mm 0.2mm 0.15mm 0.2mm 0.15mm 0.2mm 0.15mm 0.2mm 0.15mm 0.2mm 0.15mm 0.2mm"/>
 <param name="mdWireWire" value="6mil"/>
@@
 <attribute name="VALUE" x="50.927" y="54.356" size="0.8128" layer="27" rot="R180"/>
 </element>
-<element name="D1" library="diode" library_urn="urn:adsk.eagle:library:210" package="SOT23" value="10V" x="54.991" y="53.975" smashed="yes" rot="R270">
-<attribute name="NAME" x="57.912" y="53.34" size="0.8128" layer="25" font="vector" rot="R90"/>
-<attribute name="VALUE" x="52.197" y="54.864" size="0.8128" layer="27" rot="R270"/>
-</element>
 <element name="C1" library="adafruit" library_urn="urn:adsk.eagle:library:420" package="C0805" value="100nf" x="48.514" y="60.452" smashed="yes" rot="R270">
 <attribute name="NAME" x="47.879" y="62.611" size="0.8128" layer="25" font="vector"/>
@@
 <attribute name="VALUE" x="70.231" y="10.541" size="0.8128" layer="27" rot="R90"/>
 </element>
-<element name="C14" library="rcl" library_urn="urn:adsk.eagle:library:334" package="E2,5-6" value="470uf" x="63.881" y="50.165" smashed="yes" rot="R270">
-<attribute name="NAME" x="62.992" y="46.355" size="0.8128" layer="25" font="vector" ratio="10"/>
-<attribute name="VALUE" x="59.944" y="51.562" size="0.8128" layer="27" ratio="10" rot="R270"/>
-</element>
 <element name="M-OUT" library="my-custom-lib" package="7-5MM-SCREW-TERM" value="TERMINAL BLOCK 7.50MM VERT 2POS, ED110/2DS" x="94.234" y="43.688" rot="R90"/>
 <element name="PWR" library="my-custom-lib" package="7-5MM-SCREW-TERM" value="TERMINAL BLOCK 7.50MM VERT 2POS, ED110/2DS" x="49.657" y="43.053" rot="R270"/>
-<element name="C2" library="rcl" library_urn="urn:adsk.eagle:library:334" package="E2,5-6" value="470uf" x="64.008" y="12.192" smashed="yes" rot="R270">
-<attribute name="NAME" x="64.897" y="9.144" size="0.8128" layer="25" font="vector" ratio="10" rot="R180"/>
-<attribute name="VALUE" x="61.087" y="10.922" size="0.8128" layer="27" ratio="10" rot="R90"/>
-</element>
 <element name="INPUT" library="Wurth_Elektronik_Electromechanic_Terminal_Blocks_Connectors_rev16e" library_urn="urn:adsk.eagle:library:444" package="691244510004" value="5.08MM Screw Terminal, 4-POS, Wurth Elektronik PN# 691244510004" x="51.054" y="20.701" smashed="yes" rot="R90">
 <attribute name="NAME" x="57.289" y="17.76" size="1.778" layer="25" font="vector" ratio="15" rot="R270"/>
@@
 <attribute name="NAME" x="77.216" y="9.525" size="0.8128" layer="25" font="vector"/>
 <attribute name="VALUE" x="80.264" y="10.541" size="0.8128" layer="27" rot="R90"/>
+</element>
+<element name="C11" library="adafruit" library_urn="urn:adsk.eagle:library:420" package="TT5D10" value="470uf" x="63.986" y="40.212" smashed="yes">
+<attribute name="NAME" x="63.224" y="45.673" size="0.8128" layer="25" font="vector" ratio="10"/>
+<attribute name="VALUE" x="70.405" y="38.459" size="0.8128" layer="27" font="vector" ratio="10" rot="R90"/>
+</element>
+<element name="D2" library="diode" library_urn="urn:adsk.eagle:library:210" package="SMB" value="39v" x="54.991" y="53.848" smashed="yes" rot="R180">
+<attribute name="NAME" x="59.055" y="54.737" size="0.8128" layer="25" font="vector" rot="R270"/>
+<attribute name="VALUE" x="57.531" y="51.816" size="0.8128" layer="27" font="vector" rot="R180"/>
 </element>
 </elements>
@@
 <contactref element="C1" pad="2"/>
 <contactref element="C12" pad="2"/>
-<contactref element="C13" pad="2"/>
 <contactref element="C8" pad="2"/>
 <contactref element="C3" pad="2"/>
-<contactref element="C14" pad="-"/>
 <via x="67.691" y="71.755" extent="1-16" drill="0.45"/>
 <contactref element="IC1" pad="1"/>
@@
 <via x="80.01" y="42.926" extent="1-16" drill="0.45"/>
 <via x="80.01" y="40.767" extent="1-16" drill="0.45"/>
-<contactref element="C2" pad="-"/>
 <via x="69.342" y="33.02" extent="1-16" drill="0.45"/>
 <contactref element="R6" pad="1"/>
@@
 <contactref element="C7" pad="2"/>
 <contactref element="R2" pad="2"/>
-<via x="63.754" y="43.561" extent="1-16" drill="0.45"/>
-<via x="63.754" y="39.878" extent="1-16" drill="0.45"/>
-<via x="63.754" y="36.322" extent="1-16" drill="0.45"/>
+<via x="63.754" y="44.323" extent="1-16" drill="0.45"/>
+<via x="63.754" y="38.481" extent="1-16" drill="0.45"/>
+<via x="63.754" y="34.671" extent="1-16" drill="0.45"/>
 <via x="45.593" y="33.274" extent="1-16" drill="0.45"/>
 <via x="47.625" y="33.274" extent="1-16" drill="0.45"/>
@@
 <via x="89.154" y="72.898" extent="1-16" drill="0.45"/>
 <via x="98.552" y="72.898" extent="1-16" drill="0.45"/>
-<via x="63.754" y="41.783" extent="1-16" drill="0.45"/>
-<via x="63.754" y="38.1" extent="1-16" drill="0.45"/>
+<via x="63.754" y="42.418" extent="1-16" drill="0.45"/>
+<via x="63.754" y="36.576" extent="1-16" drill="0.45"/>
 <via x="49.657" y="33.274" extent="1-16" drill="0.45"/>
 <via x="53.848" y="33.274" extent="1-16" drill="0.45"/>
@@
 <via x="65.151" y="22.987" extent="1-16" drill="0.45"/>
 <via x="66.167" y="22.987" extent="1-16" drill="0.45"/>
+<contactref element="C11" pad="-"/>
+<via x="66.421" y="44.323" extent="1-16" drill="0.45"/>
+<via x="66.421" y="42.418" extent="1-16" drill="0.45"/>
+<via x="66.421" y="38.354" extent="1-16" drill="0.45"/>
+<via x="66.421" y="36.576" extent="1-16" drill="0.45"/>
+<via x="66.421" y="34.671" extent="1-16" drill="0.45"/>
+<via x="63.754" y="40.513" extent="1-16" drill="0.45"/>
 </signal>
 <signal name="OUT1" class="2">
@@
 <signal name="V+">
 <contactref element="Q1" pad="2"/>
-<contactref element="D1" pad="3"/>
 <contactref element="IC1" pad="7"/>
 <contactref element="IC2" pad="7"/>
@@
 <contactref element="C4" pad="1"/>
 <contactref element="C9" pad="1"/>
-<contactref element="C14" pad="+"/>
 <polygon width="0.3048" layer="1">
 <vertex x="55.118" y="59.182"/>
@@
 <via x="56.261" y="36.195" extent="1-16" drill="0.45"/>
 <via x="58.928" y="36.195" extent="1-16" drill="0.45"/>
-<via x="61.468" y="36.195" extent="1-16" drill="0.45"/>
-<via x="61.468" y="34.544" extent="1-16" drill="0.45"/>
 <via x="58.928" y="34.544" extent="1-16" drill="0.45"/>
 <via x="56.261" y="34.544" extent="1-16" drill="0.45"/>
-<contactref element="C2" pad="+"/>
 <wire x1="68.4969" y1="17.333" x2="68.4969" y2="15.0691" width="0.3048" layer="1"/>
 <wire x1="71.374" y1="13.423" x2="70.651" y2="13.423" width="0.3048" layer="1"/>
 <wire x1="70.651" y1="13.423" x2="69.342" y2="14.859" width="0.3048" layer="1"/>
+<contactref element="C11" pad="+"/>
+<via x="61.468" y="36.068" extent="1-16" drill="0.45"/>
+<via x="61.468" y="34.544" extent="1-16" drill="0.45"/>
+<contactref element="D2" pad="C"/>
 </signal>
 <signal name="Q1_GATE">
 <contactref element="Q1" pad="1"/>
 <contactref element="R1" pad="1"/>
-<contactref element="D1" pad="1"/>
-<polygon width="0.3048" layer="1">
-<vertex x="49.149" y="53.213"/>
+<polygon width="0.3048" layer="1">
+<vertex x="49.149" y="52.07"/>
 <vertex x="49.149" y="58.039"/>
 <vertex x="54.61" y="58.039"/>
-<vertex x="54.61" y="53.975"/>
-<vertex x="51.054" y="53.975"/>
-<vertex x="51.054" y="53.213"/>
-</polygon>
+<vertex x="54.61" y="52.07"/>
+</polygon>
+<contactref element="D2" pad="A"/>
 </signal>
 <signal name="INH_PIN">
@@
 <wire x1="65.9384" y1="62.7888" x2="62.357" y2="59.182" width="0.3048" layer="16"/>
 <wire x1="62.357" y1="59.182" x2="62.357" y2="47.752" width="0.3048" layer="16"/>
-<wire x1="62.357" y1="47.752" x2="65.405" y2="44.704" width="0.3048" layer="16"/>
-<wire x1="65.405" y1="44.704" x2="65.405" y2="28.321" width="0.3048" layer="16"/>
-<wire x1="65.405" y1="28.321" x2="63.627" y2="26.543" width="0.3048" layer="16"/>
+<wire x1="62.357" y1="47.752" x2="65.278" y2="44.831" width="0.3048" layer="16"/>
+<wire x1="65.278" y1="44.831" x2="65.278" y2="28.194" width="0.3048" layer="16"/>
+<wire x1="65.278" y1="28.194" x2="63.627" y2="26.543" width="0.3048" layer="16"/>
 <via x="63.627" y="26.543" extent="1-16" drill="0.35"/>
 <wire x1="63.627" y1="26.543" x2="63.627" y2="25.273" width="0.3048" layer="1"/>
@@
 <wire x1="65.2787125" y1="62.9419125" x2="65.278" y2="62.9419125" width="0.3048" layer="16"/>
 <wire x1="65.278" y1="62.9419125" x2="61.8998" y2="59.5637125" width="0.3048" layer="16"/>
-<wire x1="61.8998" y1="47.56261875" x2="64.9478" y2="44.51461875" width="0.3048" layer="16"/>
-<wire x1="64.9478" y1="34.2138" x2="64.389" y2="33.655" width="0.3048" layer="16"/>
+<wire x1="61.8998" y1="47.56261875" x2="64.8208" y2="44.64161875" width="0.3048" layer="16"/>
+<wire x1="64.8208" y1="34.0868" x2="64.389" y2="33.655" width="0.3048" layer="16"/>
 <wire x1="64.389" y1="33.655" x2="64.262" y2="33.655" width="0.3048" layer="16"/>
 <wire x1="64.262" y1="33.655" x2="64.135" y2="33.528" width="0.3048" layer="16"/>
@@
 <wire x1="66.797" y1="65.146" x2="66.294" y2="65.151" width="0.3048" layer="1"/>
 <wire x1="61.8998" y1="59.5637125" x2="61.8998" y2="47.56261875" width="0.3048" layer="16"/>
-<wire x1="64.9478" y1="44.51461875" x2="64.9478" y2="34.2138" width="0.3048" layer="16"/>
+<wire x1="64.8208" y1="44.64161875" x2="64.8208" y2="34.0868" width="0.3048" layer="16"/>
 </signal>
 <signal name="IN2">
