File: 20A Motor Controller.sch (EAGLE design)
At the start: 28 parts, among them IC1 BTN8962TA, IC2 BTN8962TA, Q1 FDD4141TO252

Commit message: Add files via upload
Parts:
- removed C14, C2: 470uf, rcl:CPOL-USE2.5-6
- removed D1: 10V, diode:ZENER-DIODESOT23
- added C11: 470uf, adafruit:CPOL-USTT5D10
- added D2: 39v, diode:ZENER-DIODESMB
Connections:
- net GND: now also C11.-; no longer C13.2, C14.-, C2.-
- net Q1_GATE: now also D2.A; no longer D1.A
- net V+: now also C11.+, D2.C; no longer C14.+, C2.+, D1.C
Changed lines of the file:
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@@
 <part name="P+1" library="supply1" library_urn="urn:adsk.eagle:library:371" deviceset="V+" device=""/>
 <part name="R1" library="rcl" library_urn="urn:adsk.eagle:library:334" deviceset="R-US_" device="R0805" value="10K"/>
-<part name="D1" library="diode" library_urn="urn:adsk.eagle:library:210" deviceset="ZENER-DIODE" device="SOT23" value="10V"/>
 <part name="GND1" library="supply2" library_urn="urn:adsk.eagle:library:372" deviceset="GND" device=""/>
 <part name="P+2" library="supply1" library_urn="urn:adsk.eagle:library:371" deviceset="V+" device=""/>
@@
 <part name="C13" library="adafruit" library_urn="urn:adsk.eagle:library:420" deviceset="C-US" device="C0805" value=".1uf"/>
 <part name="GND3" library="supply2" library_urn="urn:adsk.eagle:library:372" deviceset="GND" device=""/>
-<part name="GND6" library="supply2" library_urn="urn:adsk.eagle:library:372" deviceset="GND" device=""/>
 <part name="GND9" library="supply2" library_urn="urn:adsk.eagle:library:372" deviceset="GND" device=""/>
 <part name="GND10" library="supply2" library_urn="urn:adsk.eagle:library:372" deviceset="GND" device=""/>
 <part name="P+6" library="supply1" library_urn="urn:adsk.eagle:library:371" deviceset="V+" device=""/>
 <part name="P+7" library="supply1" library_urn="urn:adsk.eagle:library:371" deviceset="V+" device=""/>
-<part name="C14" library="rcl" library_urn="urn:adsk.eagle:library:334" deviceset="CPOL-US" device="E2.5-6" value="470uf"/>
-<part name="GND11" library="supply2" library_urn="urn:adsk.eagle:library:372" deviceset="GND" device=""/>
 <part name="M-OUT" library="my-custom-lib" deviceset="7-5MM-SCREW-TERM" device="" value="TERMINAL BLOCK 7.50MM VERT 2POS, ED110/2DS"/>
 <part name="PWR" library="my-custom-lib" deviceset="7-5MM-SCREW-TERM" device="" value="TERMINAL BLOCK 7.50MM VERT 2POS, ED110/2DS"/>
-<part name="C2" library="rcl" library_urn="urn:adsk.eagle:library:334" deviceset="CPOL-US" device="E2.5-6" value="470uf"/>
 <part name="GND4" library="supply2" library_urn="urn:adsk.eagle:library:372" deviceset="GND" device=""/>
 <part name="INPUT" library="Wurth_Elektronik_Electromechanic_Terminal_Blocks_Connectors_rev16e" library_urn="urn:adsk.eagle:library:444" deviceset="691244510004" device="" value="5.08MM Screw Terminal, 4-POS, Wurth Elektronik PN# 691244510004"/>
@@
 <part name="GND17" library="supply2" library_urn="urn:adsk.eagle:library:372" deviceset="GND" device=""/>
 <part name="GND18" library="supply2" library_urn="urn:adsk.eagle:library:372" deviceset="GND" device=""/>
+<part name="C11" library="adafruit" library_urn="urn:adsk.eagle:library:420" deviceset="CPOL-US" device="TT5D10" value="470uf"/>
+<part name="D2" library="diode" library_urn="urn:adsk.eagle:library:210" deviceset="ZENER-DIODE" device="SMB" value="39v"/>
 </parts>
 <sheets>
@@
 </instance>
 <instance part="GND" gate="GND" x="-58.42" y="48.26" rot="R180"/>
-<instance part="P+1" gate="1" x="-43.18" y="25.4" rot="R270"/>
+<instance part="P+1" gate="1" x="-38.1" y="25.4" rot="R270"/>
 <instance part="R1" gate="G$1" x="-58.42" y="40.64" rot="R90"/>
-<instance part="D1" gate="G$1" x="-50.8" y="33.02" rot="R270"/>
 <instance part="GND1" gate="GND" x="-73.66" y="20.32"/>
 <instance part="P+2" gate="1" x="33.02" y="48.26" rot="R270"/>
@@
 <instance part="C13" gate="G$1" x="93.98" y="45.72"/>
 <instance part="GND3" gate="GND" x="17.78" y="38.1"/>
-<instance part="GND6" gate="GND" x="93.98" y="38.1"/>
 <instance part="GND9" gate="GND" x="-58.42" y="-15.24"/>
 <instance part="GND10" gate="GND" x="-58.42" y="7.62" rot="R180"/>
 <instance part="P+6" gate="1" x="-43.18" y="7.62"/>
 <instance part="P+7" gate="1" x="-43.18" y="-15.24" rot="R180"/>
-<instance part="C14" gate="G$1" x="25.4" y="45.72"/>
-<instance part="GND11" gate="GND" x="25.4" y="38.1"/>
 <instance part="M-OUT" gate="G$1" x="-81.28" y="-5.08" rot="R180"/>
 <instance part="PWR" gate="G$1" x="-81.28" y="25.4" rot="MR0"/>
-<instance part="C2" gate="G$1" x="86.36" y="45.72"/>
-<instance part="GND4" gate="GND" x="86.36" y="38.1"/>
+<instance part="GND4" gate="GND" x="-43.18" y="15.24"/>
 <instance part="INPUT" gate="G$1" x="-83.82" y="66.04" rot="R180"/>
 <instance part="R3" gate="G$1" x="-71.12" y="60.96" rot="R180"/>
@@
 <instance part="GND17" gate="GND" x="-27.94" y="33.02"/>
 <instance part="GND18" gate="GND" x="-17.78" y="30.48"/>
+<instance part="C11" gate="G$1" x="-43.18" y="22.86"/>
+<instance part="D2" gate="G$1" x="-50.8" y="33.02" rot="R270"/>
 </instances>
 <busses>
@@
 <pinref part="Q1" gate="G$1" pin="S"/>
 <pinref part="P+1" gate="1" pin="V+"/>
-<wire x1="-45.72" y1="25.4" x2="-50.8" y2="25.4" width="0.1524" layer="91"/>
-<pinref part="D1" gate="G$1" pin="C"/>
+<wire x1="-40.64" y1="25.4" x2="-43.18" y2="25.4" width="0.1524" layer="91"/>
+<wire x1="-43.18" y1="25.4" x2="-50.8" y2="25.4" width="0.1524" layer="91"/>
 <wire x1="-50.8" y1="25.4" x2="-55.88" y2="25.4" width="0.1524" layer="91"/>
 <wire x1="-50.8" y1="25.4" x2="-50.8" y2="30.48" width="0.1524" layer="91"/>
 <junction x="-50.8" y="25.4"/>
+<pinref part="C11" gate="G$1" pin="+"/>
+<junction x="-43.18" y="25.4"/>
+<pinref part="D2" gate="G$1" pin="C"/>
 </segment>
 <segment>
 <pinref part="IC1" gate="G$1" pin="VS"/>
 <pinref part="P+2" gate="1" pin="V+"/>
-<wire x1="30.48" y1="48.26" x2="25.4" y2="48.26" width="0.1524" layer="91"/>
 <pinref part="C12" gate="G$1" pin="1"/>
-<wire x1="25.4" y1="48.26" x2="17.78" y2="48.26" width="0.1524" layer="91"/>
+<wire x1="30.48" y1="48.26" x2="17.78" y2="48.26" width="0.1524" layer="91"/>
 <wire x1="17.78" y1="48.26" x2="10.16" y2="48.26" width="0.1524" layer="91"/>
 <junction x="17.78" y="48.26"/>
-<pinref part="C14" gate="G$1" pin="+"/>
-<junction x="25.4" y="48.26"/>
 </segment>
 <segment>
@@
 <wire x1="101.6" y1="48.26" x2="93.98" y2="48.26" width="0.1524" layer="91"/>
 <pinref part="C13" gate="G$1" pin="1"/>
-<wire x1="93.98" y1="48.26" x2="86.36" y2="48.26" width="0.1524" layer="91"/>
+<wire x1="93.98" y1="48.26" x2="81.28" y2="48.26" width="0.1524" layer="91"/>
 <junction x="93.98" y="48.26"/>
-<pinref part="C2" gate="G$1" pin="+"/>
-<wire x1="86.36" y1="48.26" x2="81.28" y2="48.26" width="0.1524" layer="91"/>
-<junction x="86.36" y="48.26"/>
 </segment>
 <segment>
@@
 <pinref part="R1" gate="G$1" pin="1"/>
 <wire x1="-58.42" y1="35.56" x2="-58.42" y2="30.48" width="0.1524" layer="91"/>
-<pinref part="D1" gate="G$1" pin="A"/>
 <wire x1="-58.42" y1="35.56" x2="-50.8" y2="35.56" width="0.1524" layer="91"/>
 <junction x="-58.42" y="35.56"/>
+<pinref part="D2" gate="G$1" pin="A"/>
 </segment>
 </net>
@@
 </segment>
 <segment>
-<pinref part="C13" gate="G$1" pin="2"/>
-<pinref part="GND6" gate="GND" pin="GND"/>
-</segment>
-<segment>
 <pinref part="C8" gate="G$1" pin="2"/>
 <pinref part="GND9" gate="GND" pin="GND"/>
@@
 <pinref part="C3" gate="G$1" pin="2"/>
 <pinref part="GND10" gate="GND" pin="GND"/>
-</segment>
-<segment>
-<pinref part="C14" gate="G$1" pin="-"/>
-<pinref part="GND11" gate="GND" pin="GND"/>
 </segment>
 <segment>
@@
 </segment>
 <segment>
-<pinref part="C2" gate="G$1" pin="-"/>
-<pinref part="GND4" gate="GND" pin="GND"/>
-</segment>
-<segment>
 <pinref part="IC1" gate="G$1" pin="GND"/>
 <pinref part="GND5" gate="GND" pin="GND"/>
@@
 <pinref part="GND18" gate="GND" pin="GND"/>
 </segment>
-</net>
+<segment>
+<pinref part="GND4" gate="GND" pin="GND"/>
+<pinref part="C11" gate="G$1" pin="-"/>
+</segment>
+</net>
