File: DC Motor Controller with SLAVE OUT.brd (EAGLE design)
At the start: 57.1 x 77.1 mm, 27 parts, among them IC1 BTN8962TA, IC2 BTN8962TA, Q1 FDD4141TO252

Commit message: Add files via upload
Parts:
- removed C11: 1000uf, adafruit:TT5D10
- added C2: 470uf, adafruit:TT5D10
- added SLAVE: (no value), adafruit:1X03-CLEANBIG
- moved C6 6.21 mm to (64.5, 22.9), turned to 180 degrees
- moved R3 5.75 mm to (62.5, 28.2), turned to 180 degrees
- moved R5 3.14 mm to (64.4, 30.4)
- moved R4 3.09 mm to (64.4, 32.4)
- moved R7 2.87 mm to (64.5, 24.9), turned to 0 degrees
- moved D2 0.60 mm to (54.8, 54.4)
- moved INPUT 0.25 mm to (50.8, 20.7)
- moved PWR 0.25 mm to (49.4, 43.1)
Connections:
- net GND: now also C13.2, C2.-; no longer C11.-
- net IN1_PIN: now also SLAVE.3
- net IN2_PIN: now also SLAVE.2
- net INH_PIN: now also SLAVE.1
- net V+: now also C2.+; no longer C11.+
Routing:
- net INH_PIN: track 9.21 -> 19.0 mm
- net IN1_PIN: track 10.7 -> 20.2 mm
- net IN2_PIN: track 11.9 -> 20.5 mm
- net INH: track 55.2 -> 47.3 mm
- net IS: track 117.3 -> 124.4 mm
- net IN1: track 40.2 -> 38.6 mm
- net SR1: track 17.0 -> 15.7 mm
- net IN2: track 7.31 -> 6.10 mm
Other:
- board text added: "20A Contiunous Output / 25A Peak"
- board text added: "Brushed or Brushless DC Motor"
- board text added: "OUT"
- board text added: "Supply:"
- board text removed: "20A Continuous Output / 25A PEAK"
- board text removed: "Brushed or Brushless DC Motors"
- board text removed: "SUPPLY:"

Commit message: Add files via upload
Parts:
- C2: value 470uf -> 1000uf
Changed lines of the file:
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@@
 <attribute name="VALUE" x="62.357" y="18.288" size="1.27" layer="27" rot="R90"/>
 </element>
-<element name="C2" library="adafruit" library_urn="urn:adsk.eagle:library:420" package="TT5D10" value="470uf" x="64.0588" y="39.6494" smashed="yes">
+<element name="C2" library="adafruit" library_urn="urn:adsk.eagle:library:420" package="TT5D10" value="1000uf" x="64.0588" y="39.6494" smashed="yes">
 <attribute name="NAME" x="63.5" y="45.0342" size="0.8128" layer="25" font="vector" ratio="10"/>
 <attribute name="VALUE" x="70.3072" y="38.2016" size="0.8128" layer="27" font="vector" ratio="10" rot="R90"/>
