File: DC Motor Controller with SLAVE OUT.sch (EAGLE design)
At the start: 27 parts, among them IC1 BTN8962TA, IC2 BTN8962TA, Q1 FDD4141TO252

Commit message: Add files via upload
Parts:
- removed C11: 1000uf, adafruit:CPOL-USTT5D10
- added C2: 470uf, adafruit:CPOL-USTT5D10
- added SLAVE: (no value), adafruit:PINHD-1X3CB
Connections:
- net GND: now also C13.2, C2.-; no longer C11.-
- net IN1_PIN: now also SLAVE.3
- net IN2_PIN: now also SLAVE.2
- net INH_PIN: now also SLAVE.1
- net V+: now also C2.+; no longer C11.+
Other:
- moved on the sheet: C12, C13, R3, R5
Changed lines of the file:
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@@
 <classes>
 <class number="0" name="default" width="0.1524" drill="0.3048">
-<clearance class="0" value="0.1524"/>
+<clearance class="0" value="0.254"/>
 </class>
-<class number="1" name="GND" width="0.1524" drill="0.3048">
-<clearance class="1" value="0.1524"/>
+<class number="1" name="GND" width="0.3048" drill="0.3048">
+<clearance class="1" value="0.254"/>
 </class>
 <class number="2" name="PWR" width="0.3048" drill="0.3048">
-<clearance class="2" value="0.2032"/>
+<clearance class="2" value="0.254"/>
 </class>
 </classes>
@@
 <part name="C13" library="adafruit" library_urn="urn:adsk.eagle:library:420" deviceset="C-US" device="C0805" value=".1uf"/>
 <part name="GND3" library="supply2" library_urn="urn:adsk.eagle:library:372" deviceset="GND" device=""/>
+<part name="GND6" library="supply2" library_urn="urn:adsk.eagle:library:372" deviceset="GND" device=""/>
 <part name="GND9" library="supply2" library_urn="urn:adsk.eagle:library:372" deviceset="GND" device=""/>
 <part name="GND10" library="supply2" library_urn="urn:adsk.eagle:library:372" deviceset="GND" device=""/>
@@
 <part name="M-OUT" library="my-custom-lib" deviceset="7-5MM-SCREW-TERM" device="" value="TERMINAL BLOCK 7.50MM VERT 2POS, ED110/2DS"/>
 <part name="PWR" library="my-custom-lib" deviceset="7-5MM-SCREW-TERM" device="" value="TERMINAL BLOCK 7.50MM VERT 2POS, ED110/2DS"/>
-<part name="GND4" library="supply2" library_urn="urn:adsk.eagle:library:372" deviceset="GND" device=""/>
 <part name="INPUT" library="Wurth_Elektronik_Electromechanic_Terminal_Blocks_Connectors_rev16e" library_urn="urn:adsk.eagle:library:444" deviceset="691244510004" device="" value="5.08MM Screw Terminal, 4-POS, Wurth Elektronik PN# 691244510004"/>
 <part name="R3" library="rcl" library_urn="urn:adsk.eagle:library:334" deviceset="R-US_" device="R0805" value="10K"/>
@@
 <part name="GND17" library="supply2" library_urn="urn:adsk.eagle:library:372" deviceset="GND" device=""/>
 <part name="GND18" library="supply2" library_urn="urn:adsk.eagle:library:372" deviceset="GND" device=""/>
-<part name="C11" library="adafruit" library_urn="urn:adsk.eagle:library:420" deviceset="CPOL-US" device="TT5D10" value="1000uf"/>
+<part name="SLAVE" library="adafruit" library_urn="urn:adsk.eagle:library:420" deviceset="PINHD-1X3" device="CB"/>
+<part name="C2" library="adafruit" library_urn="urn:adsk.eagle:library:420" deviceset="CPOL-US" device="TT5D10" value="470uf"/>
+<part name="GND4" library="supply2" library_urn="urn:adsk.eagle:library:372" deviceset="GND" device=""/>
 <part name="D2" library="diode" library_urn="urn:adsk.eagle:library:210" deviceset="ZENER-DIODE" device="SMB" value="39v"/>
 </parts>
@@
 </instance>
 <instance part="GND" gate="GND" x="-58.42" y="48.26" rot="R180"/>
-<instance part="P+1" gate="1" x="-38.1" y="25.4" rot="R270"/>
+<instance part="P+1" gate="1" x="-33.02" y="25.4" rot="R270"/>
 <instance part="R1" gate="G$1" x="-58.42" y="40.64" rot="R90"/>
 <instance part="GND1" gate="GND" x="-73.66" y="20.32"/>
-<instance part="P+2" gate="1" x="33.02" y="48.26" rot="R270"/>
-<instance part="P+3" gate="1" x="104.14" y="48.26" rot="R270"/>
+<instance part="P+2" gate="1" x="25.4" y="48.26" rot="R270"/>
+<instance part="P+3" gate="1" x="93.98" y="48.26" rot="R270"/>
 <instance part="C1" gate="G$1" x="-68.58" y="35.56" rot="R180"/>
 <instance part="GND2" gate="GND" x="-68.58" y="43.18" rot="R180"/>
@@
 <instance part="C8" gate="G$1" x="-58.42" y="-7.62"/>
 <instance part="C9" gate="G$1" x="-43.18" y="-10.16" rot="R180"/>
-<instance part="C12" gate="G$1" x="17.78" y="45.72"/>
-<instance part="C13" gate="G$1" x="93.98" y="45.72"/>
-<instance part="GND3" gate="GND" x="17.78" y="38.1"/>
+<instance part="C12" gate="G$1" x="15.24" y="45.72"/>
+<instance part="C13" gate="G$1" x="86.36" y="45.72"/>
+<instance part="GND3" gate="GND" x="15.24" y="38.1"/>
+<instance part="GND6" gate="GND" x="86.36" y="38.1"/>
 <instance part="GND9" gate="GND" x="-58.42" y="-15.24"/>
 <instance part="GND10" gate="GND" x="-58.42" y="7.62" rot="R180"/>
@@
 <instance part="M-OUT" gate="G$1" x="-81.28" y="-5.08" rot="R180"/>
 <instance part="PWR" gate="G$1" x="-81.28" y="25.4" rot="MR0"/>
-<instance part="GND4" gate="GND" x="-43.18" y="15.24"/>
 <instance part="INPUT" gate="G$1" x="-83.82" y="66.04" rot="R180"/>
-<instance part="R3" gate="G$1" x="-71.12" y="60.96" rot="R180"/>
+<instance part="R3" gate="G$1" x="-63.5" y="60.96" rot="R180"/>
 <instance part="R4" gate="G$1" x="-71.12" y="76.2" rot="R180"/>
-<instance part="R5" gate="G$1" x="-71.12" y="68.58" rot="R180"/>
+<instance part="R5" gate="G$1" x="-63.5" y="68.58" rot="R180"/>
 <instance part="GND5" gate="GND" x="12.7" y="53.34" rot="R90"/>
 <instance part="GND7" gate="GND" x="83.82" y="53.34" rot="R90"/>
@@
 <instance part="GND17" gate="GND" x="-27.94" y="33.02"/>
 <instance part="GND18" gate="GND" x="-17.78" y="30.48"/>
-<instance part="C11" gate="G$1" x="-43.18" y="22.86"/>
+<instance part="SLAVE" gate="A" x="-10.16" y="0"/>
+<instance part="C2" gate="G$1" x="-40.64" y="22.86"/>
+<instance part="GND4" gate="GND" x="-40.64" y="15.24"/>
 <instance part="D2" gate="G$1" x="-50.8" y="33.02" rot="R270"/>
 </instances>
@@
 <pinref part="Q1" gate="G$1" pin="S"/>
 <pinref part="P+1" gate="1" pin="V+"/>
-<wire x1="-40.64" y1="25.4" x2="-43.18" y2="25.4" width="0.1524" layer="91"/>
-<wire x1="-43.18" y1="25.4" x2="-50.8" y2="25.4" width="0.1524" layer="91"/>
+<wire x1="-35.56" y1="25.4" x2="-40.64" y2="25.4" width="0.1524" layer="91"/>
+<wire x1="-40.64" y1="25.4" x2="-50.8" y2="25.4" width="0.1524" layer="91"/>
 <wire x1="-50.8" y1="25.4" x2="-55.88" y2="25.4" width="0.1524" layer="91"/>
 <wire x1="-50.8" y1="25.4" x2="-50.8" y2="30.48" width="0.1524" layer="91"/>
 <junction x="-50.8" y="25.4"/>
-<pinref part="C11" gate="G$1" pin="+"/>
-<junction x="-43.18" y="25.4"/>
+<pinref part="C2" gate="G$1" pin="+"/>
+<junction x="-40.64" y="25.4"/>
 <pinref part="D2" gate="G$1" pin="C"/>
 </segment>
@@
 <pinref part="P+2" gate="1" pin="V+"/>
 <pinref part="C12" gate="G$1" pin="1"/>
-<wire x1="30.48" y1="48.26" x2="17.78" y2="48.26" width="0.1524" layer="91"/>
-<wire x1="17.78" y1="48.26" x2="10.16" y2="48.26" width="0.1524" layer="91"/>
-<junction x="17.78" y="48.26"/>
+<wire x1="22.86" y1="48.26" x2="15.24" y2="48.26" width="0.1524" layer="91"/>
+<wire x1="15.24" y1="48.26" x2="10.16" y2="48.26" width="0.1524" layer="91"/>
+<junction x="15.24" y="48.26"/>
 </segment>
 <segment>
 <pinref part="IC2" gate="G$1" pin="VS"/>
 <pinref part="P+3" gate="1" pin="V+"/>
-<wire x1="101.6" y1="48.26" x2="93.98" y2="48.26" width="0.1524" layer="91"/>
+<wire x1="91.44" y1="48.26" x2="86.36" y2="48.26" width="0.1524" layer="91"/>
 <pinref part="C13" gate="G$1" pin="1"/>
-<wire x1="93.98" y1="48.26" x2="81.28" y2="48.26" width="0.1524" layer="91"/>
-<junction x="93.98" y="48.26"/>
+<wire x1="86.36" y1="48.26" x2="81.28" y2="48.26" width="0.1524" layer="91"/>
+<junction x="86.36" y="48.26"/>
 </segment>
 <segment>
@@
 </segment>
 <segment>
+<pinref part="C13" gate="G$1" pin="2"/>
+<pinref part="GND6" gate="GND" pin="GND"/>
+</segment>
+<segment>
 <pinref part="C8" gate="G$1" pin="2"/>
 <pinref part="GND9" gate="GND" pin="GND"/>
@@
 </segment>
 <segment>
+<pinref part="C2" gate="G$1" pin="-"/>
 <pinref part="GND4" gate="GND" pin="GND"/>
-<pinref part="C11" gate="G$1" pin="-"/>
 </segment>
 </net>
@@
 <pinref part="INPUT" gate="G$1" pin="2"/>
 <pinref part="R3" gate="G$1" pin="2"/>
+<wire x1="-68.58" y1="60.96" x2="-76.2" y2="60.96" width="0.1524" layer="91"/>
 <wire x1="-76.2" y1="60.96" x2="-76.2" y2="63.5" width="0.1524" layer="91"/>
 <wire x1="-76.2" y1="63.5" x2="-78.74" y2="63.5" width="0.1524" layer="91"/>
+<label x="-76.2" y="60.96" size="1.778" layer="95"/>
+</segment>
+<segment>
+<wire x1="-12.7" y1="2.54" x2="-27.94" y2="2.54" width="0.1524" layer="91"/>
+<label x="-27.94" y="2.54" size="1.778" layer="95"/>
+<pinref part="SLAVE" gate="A" pin="1"/>
 </segment>
 </net>
@@
 <wire x1="-76.2" y1="76.2" x2="-78.74" y2="76.2" width="0.1524" layer="91"/>
 <wire x1="-78.74" y1="76.2" x2="-78.74" y2="68.58" width="0.1524" layer="91"/>
+<label x="-78.74" y="71.12" size="1.778" layer="95" rot="R90"/>
+</segment>
+<segment>
+<wire x1="-27.94" y1="-2.54" x2="-12.7" y2="-2.54" width="0.1524" layer="91"/>
+<label x="-27.94" y="-2.54" size="1.778" layer="95"/>
+<pinref part="SLAVE" gate="A" pin="3"/>
 </segment>
 </net>
@@
 <pinref part="INPUT" gate="G$1" pin="3"/>
 <pinref part="R5" gate="G$1" pin="2"/>
+<wire x1="-68.58" y1="68.58" x2="-76.2" y2="68.58" width="0.1524" layer="91"/>
 <wire x1="-76.2" y1="68.58" x2="-76.2" y2="66.04" width="0.1524" layer="91"/>
 <wire x1="-76.2" y1="66.04" x2="-78.74" y2="66.04" width="0.1524" layer="91"/>
+<label x="-76.2" y="68.58" size="1.778" layer="95"/>
+</segment>
+<segment>
+<wire x1="-12.7" y1="0" x2="-27.94" y2="0" width="0.1524" layer="91"/>
+<label x="-27.94" y="0" size="1.778" layer="95"/>
+<pinref part="SLAVE" gate="A" pin="2"/>
 </segment>
 </net>
@@
 </segment>
 <segment>
-<wire x1="-60.96" y1="60.96" x2="-66.04" y2="60.96" width="0.1524" layer="91"/>
+<wire x1="-50.8" y1="60.96" x2="-58.42" y2="60.96" width="0.1524" layer="91"/>
 <pinref part="R3" gate="G$1" pin="1"/>
-<label x="-66.04" y="60.96" size="1.778" layer="95"/>
+<label x="-55.88" y="60.96" size="1.778" layer="95"/>
 </segment>
 </net>
@@
 </segment>
 <segment>
-<wire x1="-66.04" y1="68.58" x2="-60.96" y2="68.58" width="0.1524" layer="91"/>
+<wire x1="-58.42" y1="68.58" x2="-50.8" y2="68.58" width="0.1524" layer="91"/>
 <pinref part="R5" gate="G$1" pin="1"/>
-<label x="-66.04" y="68.58" size="1.778" layer="95"/>
-</segment>
-</net>
+<label x="-55.88" y="68.58" size="1.778" layer="95"/>
+</segment>
+</net>

Commit message: Add files via upload
Parts:
- C2: value 470uf -> 1000uf
Changed lines of the file:
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@@
 <part name="GND18" library="supply2" library_urn="urn:adsk.eagle:library:372" deviceset="GND" device=""/>
 <part name="SLAVE" library="adafruit" library_urn="urn:adsk.eagle:library:420" deviceset="PINHD-1X3" device="CB"/>
-<part name="C2" library="adafruit" library_urn="urn:adsk.eagle:library:420" deviceset="CPOL-US" device="TT5D10" value="470uf"/>
+<part name="C2" library="adafruit" library_urn="urn:adsk.eagle:library:420" deviceset="CPOL-US" device="TT5D10" value="1000uf"/>
 <part name="GND4" library="supply2" library_urn="urn:adsk.eagle:library:372" deviceset="GND" device=""/>
 <part name="D2" library="diode" library_urn="urn:adsk.eagle:library:210" deviceset="ZENER-DIODE" device="SMB" value="39v"/>
